Commit message: lidar

File: description/lidar.xacro (robot description, xacro)
@@ -4,5 +4,5 @@
         <parent link="chassis"/>
         <child link="laser_frame"/>
-        <origin xyz="0.122 0 0.212" rpy="0 0 0"/>
+        <origin xyz="0.0 0 0.5" rpy="0 0 0"/>
     </joint>
     <link name="laser_frame">

File: description/ros2_control.xacro (robot description, xacro)
@@ -8,5 +8,5 @@
                 <param name="right_wheel_name">right_wheel_joint</param>
                 <param name="loop_rate">30</param>
-                <param name="device">/dev/ttyUSB0</param>
+                <param name="device">/dev/serial/by-path/platform-fd500000.pcie-pci-0000:01:00.0-usb-0:1.4:1.0-port0</param>
                 <param name="baud_rate">57600</param>
                 <param name="timeout_ms">1000</param>

Commit message: lidar

File: description/lidar.xacro (robot description, xacro)
@@ -4,10 +4,10 @@
         <parent link="chassis"/>
         <child link="laser_frame"/>
-        <origin xyz="0.0 0 0.5" rpy="0 0 0"/>
+        <origin xyz="0.09 0 0.141" rpy="0 0 0"/>
     </joint>
     <link name="laser_frame">
         <visual>
             <geometry>
-                <cylinder radius="0.05" length="0.04"/>
+                <cylinder radius="0.05" length="0.03"/>
             </geometry>
             <material name="black"/>
@@ -22,8 +22,8 @@
         <collision>
             <geometry>
-                <cylinder radius="0.05" length="0.04"/>
+                <cylinder radius="0.05" length="0.03"/>
             </geometry>
         </collision>
-        <xacro:inertial_cylinder mass="0.1" length="0.04" radius="0.05">
+        <xacro:inertial_cylinder mass="0.1" length="0.04" radius="0.03">
             <origin xyz="0 0 0" rpy="0 0 0"/>
         </xacro:inertial_cylinder>

File: description/robot.urdf.xacro (robot description, xacro)
@@ -10,5 +10,5 @@
         <xacro:include filename="gazebo_control.xacro" />
     </xacro:unless>
-    <!-- <xacro:include filename="lidar.xacro" /> -->
+    <xacro:include filename="lidar.xacro" />
     <xacro:include filename="camera.xacro" />
     <!-- <xacro:include filename="depth_camera.xacro" /> -->

File: description/robot_core.xacro (robot description, xacro)
@@ -4,13 +4,13 @@
     <xacro:property name="chassis_length" value="0.18"/>
     <xacro:property name="chassis_width" value="0.18"/>
-    <xacro:property name="chassis_height" value="0.12"/>
+    <xacro:property name="chassis_height" value="0.116"/>
     <xacro:property name="chassis_mass" value="1.0"/>
     <xacro:property name="wheel_radius" value="0.035"/>
     <xacro:property name="wheel_thickness" value="0.028"/>
     <xacro:property name="wheel_mass" value="0.05"/>
-    <xacro:property name="wheel_offset_x" value="0.13"/>
+    <xacro:property name="wheel_offset_x" value="0.128"/>
     <xacro:property name="wheel_offset_y" value="0.11"/>
-    <xacro:property name="wheel_offset_z" value="0.027"/>
-    <xacro:property name="caster_wheel_radius" value="0.01"/>
+    <xacro:property name="wheel_offset_z" value="0.019"/>
+    <xacro:property name="caster_wheel_radius" value="0.014"/>
     <xacro:property name="caster_wheel_mass" value="0.01"/>
     <xacro:property name="caster_wheel_offset_x" value="0.02"/>
