Commit message: camera

File: description/camera.xacro (robot description, xacro)
@@ -4,5 +4,5 @@
         <parent link="chassis"/>
         <child link="camera_link"/>
-        <origin xyz="0.18 0 0.09" rpy="0 0 0"/>
+        <origin xyz="0.18 0 0.083" rpy="0 0 0"/>
     </joint>
     <link name="camera_link">
@@ -27,9 +27,10 @@
             <update_rate>10</update_rate>
             <camera>
-                <horizontal_fov>1.089</horizontal_fov>
+                <!-- <horizontal_fov>1.089</horizontal_fov> -->
+                <horizontal_fov>2.792</horizontal_fov>
                 <image>
                     <format>R8G8B8</format>
-                    <width>640</width>
-                    <height>480</height>
+                    <width>1280</width>
+                    <height>720</height>
                 </image>
                 <clip>
